Commit message: Update common_properties.xacro

File: my_robot/urdf/common_properties.xacro (robot description, xacro)
@@ -6,4 +6,10 @@
     <material name="grey">
         <color rgba=" 0.5 0.5 0.5 1 "/>
+    </material>
+    <material name="orange">
+        <color rgba="1.0 0.65 0.0 1"/>
+    </material>
+    <material name="yellow">
+        <color rgba="1.0 1.0 0.0 1"/>
     </material>
     <xacro:macro name="box_inertia" params="m l w h xyz rpy">
