Commit message: Update mobile_base_gazebo.xacro

File: my_robot/urdf/mobile_base_gazebo.xacro (robot description, xacro)
@@ -1,18 +1,35 @@
 <?xml version="1.0"?>
-<robot xmlns:xacro="http://www.ros.org/wiki/xacro">
-    <!--gazebo>
-        <plugin name="diff_drive_control" filename="ignition-gazebo-diff-drive-system">
-            <update_rate>50</update_rate>
-            <left_joint>base_left_wheel</left_joint>
-            <right_joint>base_right_wheel</right_joint>
+<robot xmlns:xacro="http://www.ros.org/wiki/xacro" name="my_robot" >
+    <!-- Gazebo plugin for differential drive -->
+    <gazebo>
+        <plugin filename="gz-sim-diff-drive-system" name="gz::sim::systems::DiffDrive">
+            <odom_publisher_frequency>50</odom_publisher_frequency>
+            <left_joint>base_right_wheel</left_joint>
+            <right_joint>base_left_wheel</right_joint>
             <wheel_separation>0.45</wheel_separation>
-            <wheel_diameter>0.2</wheel_diameter>
+            <wheel_diameter>0.1</wheel_diameter>
+            <max_wheel_torque>20</max_wheel_torque>
+            <max_linear_acceleration>5.0</max_linear_acceleration>
+            <topic>cmd_vel</topic>
             <publish_odom>true</publish_odom>
             <publish_odom_tf>true</publish_odom_tf>
             <publish_wheel_tf>true</publish_wheel_tf>
-            <odometry_topic>odom</odometry_topic>
-            <odometry_frame>odom</odometry_frame>
-            <robot_base_frame>base_footprint</robot_base_frame>
+            <odom_topic>odom</odom_topic>
+            <frame_id>odom</frame_id>
+            <child_frame_id>base_link</child_frame_id>
         </plugin>
-    </gazebo-->
+        <plugin filename="gz-sim-joint-state-publisher-system" name="gz::sim::systems::JointStatePublisher">
+            <update_rate>50</update_rate>
+            <joint_name>base_right_wheel</joint_name>
+            <joint_name>base_left_wheel</joint_name>
+        </plugin>
+    </gazebo>
+    <gazebo reference="base_link">
+        <material>Gazebo/Blue</material>
+    </gazebo>
+    <gazebo reference="caster_wheel_link">
+        <material>Gazebo/Grey</material>
+        <mu1>0.1</mu1>
+        <mu2>0.2</mu2>
+    </gazebo>
 </robot>
