Commit message: Update camera.xacro

File: my_robot/urdf/camera.xacro (robot description, xacro)
@@ -1,12 +1,7 @@
 <?xml version="1.0"?>
-<robot xmlns:xacro="http://www.ros.org/wiki/xacro" name="my_robot">
-    <!-- Camera dimensions -->
+<robot xmlns:xacro="http://ros.org/wiki/xacro" name="my_robot">
     <xacro:property name="camera_length" value="0.01"/>
     <xacro:property name="camera_height" value="0.05"/>
     <xacro:property name="camera_width" value="0.1"/>
-    <!-- Ensure base dimensions exist -->
-    <xacro:property name="base_length" value="0.6"/>
-    <xacro:property name="base_height" value="0.2"/>
-    <!-- Camera link -->
     <link name="camera_link">
         <visual>
@@ -14,5 +9,7 @@
                 <box size="${camera_length} ${camera_width} ${camera_height}" />
             </geometry>
-            <material name="grey"/>
+            <material name="Grey">
+                <color rgba="0.5 0.5 0.5 1.0"/>
+            </material>
         </visual>
         <collision>
@@ -22,42 +19,19 @@
         </collision>
         <xacro:box_inertia m="0.1" l="${camera_length}" w="${camera_width}" h="${camera_height}"
-                            xyz="0 0 0"  rpy="0 0 0"/>
+                            xyz="0 0 0" rpy="0 0 0" />
     </link>
-    <!-- Joint to attach the camera to the base -->
     <joint name="base_camera_joint" type="fixed">
         <parent link="base_link"/>
         <child link="camera_link" />
-        <origin xyz="${(base_length + camera_length)/2.0} 0 ${base_height / 2.0}" rpy="0 0 0"/>
+        <origin xyz="${(base_length + camera_length) / 2.0} 0 ${base_height / 2.0}" rpy="0 0 0"/>
     </joint>
-    <!-- Ignition Gazebo camera plugin -->
     <gazebo reference="camera_link">
-        <sensor name="camera_sensor" type="camera">
-            <camera>
-                <horizontal_fov>1.047</horizontal_fov> <!-- 60 degrees -->
-                <image>
-                    <width>640</width>
-                    <height>480</height>
-                    <format>R8G8B8</format>
-                </image>
-                <clip>
-                    <near>0.1</near>
-                    <far>100</far>
-                </clip>
-            </camera>
-            <!-- Noise should be here -->
-            <noise>
-                <type>gaussian</type>
-                <mean>0.0</mean>
-                <stddev>0.007</stddev>
-            </noise>
-            <always_on>true</always_on>
+        <material>Gazebo/Red</material>
+        <sensor name="camera_sensor" type="camera" >
+            <pose>0 0 0.05 0 0 0</pose>
             <update_rate>10</update_rate>
-            <visualize>true</visualize>
-            <topic>camera/image_raw</topic>
-            <plugin filename="libgz-sim-sensor-system.so" name="gz::sim::systems::Camera">
-                <ros>
-                    <namespace>/</namespace>
-                    <remapping>camera/image_raw:=camera/image_raw</remapping>
-                </ros>
+            <visualize>false</visualize>
+            <plugin name="camera_controller" filename="libgazebo_ros_camera.so">
+                <frame_name>camera_link</frame_name>
             </plugin>
         </sensor>

Commit message: Update camera.xacro

File: my_robot/urdf/camera.xacro (robot description, xacro)
@@ -38,2 +38,64 @@
     </gazebo>
 </robot>
+<?xml version="1.0"?>
+<robot xmlns:xacro="http://www.ros.org/wiki/xacro" name="my_robot">
+    <xacro:property name="lidar_radius" value="0.1"/>
+    <xacro:property name="lidar_length" value="0.09"/>
+    <link name="lidar_link">
+        <visual>
+            <geometry>
+                <cylinder radius="${lidar_radius}" length="${lidar_length}"/>
+            </geometry>
+            <origin xyz="0.0 0.0 0.0" rpy="0.0 0.0 0.0"/>
+            <material name="red"/>
+        </visual>
+        <collision>
+            <geometry>
+                <cylinder radius="${lidar_radius}" length="${lidar_length}"/>
+            </geometry>
+            <origin xyz="0.0 0.0 0.0" rpy="0.0 0.0 0.0"/>
+        </collision>
+            <xacro:cylinder_inertia  m="0.2" r="${lidar_radius}" h="${lidar_length}"
+                                    xyz="0 0 0" rpy="0 0 0" />
+    </link>
+    <joint name="base_lidar_joint" type="fixed">
+        <parent link="base_link"/>
+        <child link="lidar_link"/>
+        <origin xyz="0.0 0.0 ${base_height}" rpy="0.0 0.0 0.0"/>
+    </joint>
+    <gazebo reference="lidar_link">
+        <material>Gazebo/Red</material>
+        <sensor name="lidar_sensor" type="ray">
+            <visualize>true</visualize>
+            <pose>0 0 0 0 0 0</pose>
+            <update_rate>20</update_rate>
+            <ray>
+                <scan>
+                    <horizontal>
+                        <samples>360</samples>
+                        <resolution>1</resolution>
+                        <min_angle>-3.14159</min_angle>
+                        <max_angle>3.14159</max_angle>
+                    </horizontal>
+                </scan>
+                <range>
+                    <min>0.1</min>
+                    <max>10.0</max>
+                    <resolution>0.01</resolution>
+                </range>
+                <!--<noise>
+                    <type>gaussian</type>
+                    <mean>0.0</mean>
+                    <stddev>0.01</stddev>
+                </noise>-->
+            </ray>
+            <plugin name="laser_controller" filename="libgazebo_ros_ray_sensor.so">
+                <ros>
+                    <argument>~/out:=scan</argument>
+                </ros>
+                <output_type>sensor_msgs/LaserScan</output_type>
+                <frameName>lidar_link</frameName>
+            </plugin>
+        </sensor>
+    </gazebo>
+</robot>
